File: KICAD/BoardV2/BoardV1/ConConversor.kicad_pcb (KiCad board)
At the start: 2 copper layers, 72.4 x 48.3 mm, 104 parts, among them IC1 STM8S103F3P3, J1 DHT11, J10 ARRIBA_I, J11 ARRIBA_D, J12 ABAJO_D, J13 ABAJO_I, J2 UART, J3 SWIM, J4 USB_B_Micro, J5 RS485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

Commit message: 20211101
Parts:
- moved J4 2.35 mm to (71.3, 94.7)
Routing:
- net 5VGND: track 463.2 -> 471.6 mm, vias 28 -> 29
- net 5V: track 109.0 -> 116.3 mm
- removed copper zone on B.Cu, net (none)
Other:
- outline, holes or cut-outs redrawn
